File: GP2040-CE Tester/Mega2560.kicad_sch (KiCad schematic)
At the start: 0 parts

Commit message: adding most of the components, and schematic connections
Parts:
- added C24, C25, C27, C28, C29, C30: 100nF, Capacitor_SMD:C_0603_1608Metric, symbol Device:C
- added C26: 1μF, Capacitor_SMD:C_0603_1608Metric, symbol Device:C
- added D1, D2: LED, LED_SMD:LED_0603_1608Metric, symbol Device:LED
- added JP1: Jumper_2_Open, Jumper:SolderJumper-2_P1.3mm_Open_TrianglePad1.0x1.5mm, symbol Jumper:Jumper_2_Open
- added L1: 10uH, Inductor_SMD:L_0603_1608Metric, symbol Device:L
- added R13, R14, R20, R21: 22R, Resistor_SMD:R_0603_1608Metric, symbol Device:R
- added R15, R16, R17, R18, R19: 1K, Resistor_SMD:R_0603_1608Metric, symbol Device:R
- added U7: ATmega2560-16A, Package_QFP:TQFP-100_14x14mm_P0.5mm, symbol MCU_Microchip_ATmega:ATmega2560-16A
- added U8: ATmega16U2-M, Package_DFN_QFN:QFN-32-1EP_5x5mm_P0.5mm_EP3.1x3.1mm, symbol MCU_Microchip_ATmega:ATmega16U2-M
- added U9: MAX3421EEHJ+T, GP2040-CE-Tester:MAX3421EEHJ+T, symbol GP2040-CE-Tester:MAX3421EEHJ+T
- added Y1, Y2: SIT9003AC-24-33ED-16.00000T, GP2040-CE-Tester:SIT9003AC-24-33ED-16.00000T, symbol GP2040-CE-Tester:SIT9003AC-24-33ED-16.00000T
Connections:
- new net: R17.1, U8.8 (PD2)
- new net: R21.1, U9.20 (D-)
- new net: C25.1, R19.1, U8.13 (~{HWB}/PD7)
- new net: D1.2 (A), R15.1
- new net: R14.2, U8.30 (D-)
- new net: R20.1, U9.21 (D+)
- new net: D2.2 (A), R16.1
- new net: U7.34 (XTAL1), Y2.3 (CLK)
- new net: R13.1, U8.29 (D+)
- new net: R18.1, U8.9 (PD3)
- new net: U8.1 (XTAL1), Y1.3 (CLK)
- new net: C26.1, U8.27 (UCAP)
- new net +3.3V: Y1.4 (VDD), Y2.4 (VDD)
- new net +5V: C24.1, C27.1, C28.1, C29.1, L1.1, R15.2, R16.2, U7.10 (VCC), U7.31 (VCC), U7.61 (VCC), U7.80 (VCC), U8.31 (UVCC), U8.32 (AVCC), U8.4 (VCC)
- new net AVCC: C30.1, L1.2, U7.100 (AVCC)
- new net GND: C24.2, C26.2, C27.2, C28.2, C29.2, C30.2, R19.2, U7.11 (GND), U7.32 (GND), U7.62 (GND), U7.81 (GND), U7.99 (GND), U8.28 (UGND), U8.3 (GND), U8.33 (GND), Y1.2 (GND), Y2.2 (GND)
- new net MEGA_USB_D+: R13.2
- new net MEGA_USB_D-: R14.1
- new net PE0: R18.2, U7.2 (PE0)
- new net PE1: R17.2, U7.3 (PE1)
- new net RESET: C25.2, JP1.1 (A), JP1.2 (B), U7.30 (~{RESET})
- new net RXL: D2.1 (K), U8.10 (PD4)
- new net SHIELDUSBD+: R20.2
- new net SHIELDUSBD-: R21.2
- new net TXL: D1.1 (K), U8.11 (PD5)
- no-connect marks 0 -> 11
