File: GP2040-CE Tester/PowerManagement.kicad_sch (KiCad schematic)
At the start: 0 parts

Commit message: adding most of the components, and schematic connections
Parts:
- added C13, C14: 10uF, Capacitor_SMD:C_0603_1608Metric, symbol Device:C
- added U4: NCP1117-3.3_SOT223, Package_TO_SOT_SMD:SOT-223-3_TabPin2, symbol Regulator_Linear:NCP1117-3.3_SOT223
Connections:
- new net +3.3V: C14.1, U4.2 (VO)
- new net GND: C13.2, C14.2, U4.1 (GND)
- new net VBUS: C13.1, U4.3 (VI)
Changed lines of the file:
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@@
 (kicad_sch (version 20230121) (generator eeschema)
   (paper "A4")
+  (junction (at 64.77 30.48) (diameter 0) (color 0 0 0 0)
+  )
+  (junction (at 34.29 30.48) (diameter 0) (color 0 0 0 0)
+  )
+  (wire (pts (xy 64.77 30.48) (xy 69.85 30.48))
+    (stroke (width 0) (type default))
+  )
+  (wire (pts (xy 34.29 30.48) (xy 44.45 30.48))
+    (stroke (width 0) (type default))
+  )
+  (wire (pts (xy 59.69 30.48) (xy 64.77 30.48))
+    (stroke (width 0) (type default))
+  )
+  (wire (pts (xy 25.4 30.48) (xy 34.29 30.48))
+    (stroke (width 0) (type default))
+  )
+  (hierarchical_label "3v3" (shape input) (at 69.85 30.48 0) (fields_autoplaced)
+    (effects (font (size 1.27 1.27)) (justify left))
+  )
+  (hierarchical_label "VBUS" (shape input) (at 25.4 30.48 270) (fields_autoplaced)
+    (effects (font (size 1.27 1.27)) (justify right))
+  )
+  (symbol (lib_id "power:VBUS") (at 25.4 30.48 0) (unit 1)
+    (in_bom yes) (on_board yes) (dnp no) (fields_autoplaced)
+    (property "Reference" "#PWR015" (at 25.4 34.29 0)
+      (effects (font (size 1.27 1.27)) hide)
+    )
+    (property "Value" "VBUS" (at 25.4 26.67 0)
+      (effects (font (size 1.27 1.27)))
+    )
+    (property "Footprint" "" (at 25.4 30.48 0)
+      (effects (font (size 1.27 1.27)) hide)
+    )
+    (property "Datasheet" "" (at 25.4 30.48 0)
+      (effects (font (size 1.27 1.27)) hide)
+    )
+    (pin "1")
+    (instances
+      (project "GP2040-CE Tester"
+        (path "/7572bcd0-c27e-4c00-81c9-62cf732047bc/808745e8-dff6-4b0f-a972-b91efdddf17c"
+          (reference "#PWR015") (unit 1)
+        )
+      )
+    )
+  )
+  (symbol (lib_id "Device:C") (at 64.77 34.29 0) (unit 1)
+    (in_bom yes) (on_board yes) (dnp no) (fields_autoplaced)
+    (property "Reference" "C14" (at 68.58 33.655 0)
+      (effects (font (size 1.27 1.27)) (justify left))
+    )
+    (property "Value" "10uF" (at 68.58 36.195 0)
+      (effects (font (size 1.27 1.27)) (justify left))
+    )
+    (property "Footprint" "Capacitor_SMD:C_0603_1608Metric" (at 65.7352 38.1 0)
+      (effects (font (size 1.27 1.27)) hide)
+    )
+    (property "Datasheet" "~" (at 64.77 34.29 0)
+      (effects (font (size 1.27 1.27)) hide)
+    )
+    (pin "1")
+    (pin "2")
+    (instances
+      (project "GP2040-CE Tester"
+        (path "/7572bcd0-c27e-4c00-81c9-62cf732047bc/808745e8-dff6-4b0f-a972-b91efdddf17c"
+          (reference "C14") (unit 1)
+        )
+      )
+    )
+  )
+  (symbol (lib_id "power:GND") (at 52.07 38.1 0) (unit 1)
+    (in_bom yes) (on_board yes) (dnp no) (fields_autoplaced)
+    (property "Reference" "#PWR017" (at 52.07 44.45 0)
+      (effects (font (size 1.27 1.27)) hide)
+    )
+    (property "Value" "GND" (at 52.07 43.18 0)
+      (effects (font (size 1.27 1.27)))
+    )
+    (property "Footprint" "" (at 52.07 38.1 0)
+      (effects (font (size 1.27 1.27)) hide)
+    )
+    (property "Datasheet" "" (at 52.07 38.1 0)
+      (effects (font (size 1.27 1.27)) hide)
+    )
+    (pin "1")
+    (instances
+      (project "GP2040-CE Tester"
+        (path "/7572bcd0-c27e-4c00-81c9-62cf732047bc/808745e8-dff6-4b0f-a972-b91efdddf17c"
+          (reference "#PWR017") (unit 1)
+        )
+      )
+    )
+  )
+  (symbol (lib_id "Device:C") (at 34.29 34.29 0) (unit 1)
+    (in_bom yes) (on_board yes) (dnp no) (fields_autoplaced)
+    (property "Reference" "C13" (at 38.1 33.655 0)
+      (effects (font (size 1.27 1.27)) (justify left))
+    )
+    (property "Value" "10uF" (at 38.1 36.195 0)
+      (effects (font (size 1.27 1.27)) (justify left))
+    )
+    (property "Footprint" "Capacitor_SMD:C_0603_1608Metric" (at 35.2552 38.1 0)
+      (effects (font (size 1.27 1.27)) hide)
+    )
+    (property "Datasheet" "~" (at 34.29 34.29 0)
+      (effects (font (size 1.27 1.27)) hide)
+    )
+    (pin "1")
+    (pin "2")
+    (instances
+      (project "GP2040-CE Tester"
+        (path "/7572bcd0-c27e-4c00-81c9-62cf732047bc/808745e8-dff6-4b0f-a972-b91efdddf17c"
+          (reference "C13") (unit 1)
+        )
+      )
+    )
+  )
+  (symbol (lib_id "power:GND") (at 34.29 38.1 0) (unit 1)
+    (in_bom yes) (on_board yes) (dnp no) (fields_autoplaced)
+    (property "Reference" "#PWR016" (at 34.29 44.45 0)
+      (effects (font (size 1.27 1.27)) hide)
+    )
+    (property "Value" "GND" (at 34.29 43.18 0)
+      (effects (font (size 1.27 1.27)))
+    )
+    (property "Footprint" "" (at 34.29 38.1 0)
+      (effects (font (size 1.27 1.27)) hide)
+    )
+    (property "Datasheet" "" (at 34.29 38.1 0)
+      (effects (font (size 1.27 1.27)) hide)
+    )
+    (pin "1")
+    (instances
+      (project "GP2040-CE Tester"
+        (path "/7572bcd0-c27e-4c00-81c9-62cf732047bc/808745e8-dff6-4b0f-a972-b91efdddf17c"
+          (reference "#PWR016") (unit 1)
+        )
+      )
+    )
+  )
+  (symbol (lib_id "power:+3.3V") (at 69.85 30.48 0) (unit 1)
+    (in_bom yes) (on_board yes) (dnp no) (fields_autoplaced)
+    (property "Reference" "#PWR018" (at 69.85 34.29 0)
+      (effects (font (size 1.27 1.27)) hide)
+    )
+    (property "Value" "+3.3V" (at 69.85 26.67 0)
+      (effects (font (size 1.27 1.27)))
+    )
+    (property "Footprint" "" (at 69.85 30.48 0)
+      (effects (font (size 1.27 1.27)) hide)
+    )
+    (property "Datasheet" "" (at 69.85 30.48 0)
+      (effects (font (size 1.27 1.27)) hide)
+    )
+    (pin "1")
+    (instances
+      (project "GP2040-CE Tester"
+        (path "/7572bcd0-c27e-4c00-81c9-62cf732047bc/808745e8-dff6-4b0f-a972-b91efdddf17c"
+          (reference "#PWR018") (unit 1)
+        )
+      )
+    )
+  )
+  (symbol (lib_id "Regulator_Linear:NCP1117-3.3_SOT223") (at 52.07 30.48 0) (unit 1)
+    (in_bom yes) (on_board yes) (dnp no) (fields_autoplaced)
+    (property "Reference" "U4" (at 52.07 24.13 0)
+      (effects (font (size 1.27 1.27)))
+    )
+    (property "Value" "NCP1117-3.3_SOT223" (at 52.07 26.67 0)
+      (effects (font (size 1.27 1.27)))
+    )
+    (property "Footprint" "Package_TO_SOT_SMD:SOT-223-3_TabPin2" (at 52.07 25.4 0)
+      (effects (font (size 1.27 1.27)) hide)
+    )
+    (property "Datasheet" "http://www.onsemi.com/pub_link/Collateral/NCP1117-D.PDF" (at 54.61 36.83 0)
+      (effects (font (size 1.27 1.27)) hide)
+    )
+    (pin "1")
+    (pin "2")
+    (pin "3")
+    (instances
+      (project "GP2040-CE Tester"
+        (path "/7572bcd0-c27e-4c00-81c9-62cf732047bc/808745e8-dff6-4b0f-a972-b91efdddf17c"
+          (reference "U4") (unit 1)
+        )
+      )
+    )
+  )
+  (symbol (lib_id "power:GND") (at 64.77 38.1 0) (unit 1)
+    (in_bom yes) (on_board yes) (dnp no) (fields_autoplaced)
+    (property "Reference" "#PWR019" (at 64.77 44.45 0)
+      (effects (font (size 1.27 1.27)) hide)
+    )
+    (property "Value" "GND" (at 64.77 43.18 0)
+      (effects (font (size 1.27 1.27)))
+    )
+    (property "Footprint" "" (at 64.77 38.1 0)
+      (effects (font (size 1.27 1.27)) hide)
+    )
+    (property "Datasheet" "" (at 64.77 38.1 0)
+      (effects (font (size 1.27 1.27)) hide)
+    )
+    (pin "1")
+    (instances
+      (project "GP2040-CE Tester"
+        (path "/7572bcd0-c27e-4c00-81c9-62cf732047bc/808745e8-dff6-4b0f-a972-b91efdddf17c"
+          (reference "#PWR019") (unit 1)
+        )
+      )
+    )
+  )
 )
