File: Dueling Picos/Dueling Picos.kicad_pcb (KiCad board)
At the start: 2 copper layers, 72.8 x 58.3 mm, 4 parts, among them J1 USB_A, J2 Conn_01x04_Pin, U1 Host Pico, U2 GP2040-CE Pico

Commit message: syncing
Parts:
- added R1: 22R, Resistor_SMD:R_0201_0603Metric, F.Cu at (114.7, 56.3)
- added R2: 22R, Resistor_SMD:R_0201_0603Metric, F.Cu at (115.5, 56.3)
- J1: value USB_A -> UJ2-AH-4-TH; footprint Connector_USB:USB_A_Molex_67643_Horizontal -> UJ2-AH-4-TH:CUI_UJ2-AH-4-TH
Connections:
- U1 pad 1: /D+ -> /+
- U1 pad 2: /D- -> /-
- U1 pad 38: GND -> unconnected-(U1-GND-Pad38)
Routing:
- net /-: track 0.00 -> 8.70 mm
- net /+: track 0.00 -> 8.55 mm
- net /D-: track 24.2 -> 17.5 mm
- net /D+: track 24.1 -> 17.4 mm
Other:
- board text added: "3V3"
- board text added: "3V3_EN"
- board text added: "ADC_VREF"
- board text added: "AGND"
- board text added: "D+"
- board text added: "D-"
- board text added: "GND"
- board text added: "GP0"
- board text added: "GP1"
- board text added: "GP10"
- board text added: "GP11"
- board text added: "GP12"
- board text added: "GP13"
- board text added: "GP14"
- board text added: "GP15"
- board text added: "GP16"
- board text added: "GP17"
- board text added: "GP18"
- board text added: "GP19"
- board text added: "GP2"
- board text added: "GP20"
- board text added: "GP2040-CE Pico"
- board text added: "GP21"
- board text added: "GP22"
- board text added: "GP26"
- board text added: "GP27"
- board text added: "GP28"
- board text added: "GP3"
- board text added: "GP4"
- board text added: "GP5"
- board text added: "GP6"
- board text added: "GP7"
- board text added: "GP8"
- board text added: "GP9"
- board text added: "Host Pico"
- board text added: "Host Pico will run the latency tests. You will need to connect the GP2040-CE Pico to the USB-A port connected to the Host Pico."
- board text added: "RUN"
- board text added: "SWCLK"
- board text added: "SWDIO"
- board text added: "Shield"
- board text added: "VBUS"
- board text added: "VSYS"
