File: Dueling Picos/Dueling Picos.kicad_sch (KiCad schematic)
At the start: 4 parts, among them J1 USB_A, J2 Conn_01x04_Pin, U1 Host Pico, U2 GP2040-CE Pico

Commit message: syncing
Parts:
- added R1, R2: 22R, Resistor_SMD:R_0201_0603Metric, symbol Device:R
- J1: value USB_A -> UJ2-AH-4-TH; footprint Connector_USB:USB_A_Molex_67643_Horizontal -> UJ2-AH-4-TH:CUI_UJ2-AH-4-TH; symbol Connector:USB_A -> UJ2-AH-4-TH:UJ2-AH-4-TH; MANUFACTURER (none) -> CUI INC; PART_REV (none) -> 1.0; STANDARD (none) -> MANUFACTURER RECOMMENDATIONS
Connections:
- net D+: now also R1.1; no longer U1.1 (GPIO0)
- net D-: now also R2.1; no longer U1.2 (GPIO1)
- net GND: no longer J1.5 (Shield), U1.38 (GND)
- new net +: R1.2, U1.1 (GPIO0)
- new net -: R2.2, U1.2 (GPIO1)
- new net Earth: J1.SH1 (SHIELD), J1.SH2 (SHIELD__1)
